Commit message: ball_manipulation with weighted CLIK

File: model/irc_man.urdf (robot description, URDF)
Before this commit: robot irc_man, 11 links, 10 joints
Joints:
- joint ee: origin xyz=0.0001 -0.0205 -0.18185 rpy=0 0 0 -> xyz=0.0001 -0.0205 -0.15 rpy=0 0 0

Commit message: feat: pick_sequence great

File: model/irc_man.urdf (robot description, URDF)
Before this commit: robot irc_man, 11 links, 10 joints
Joints:
- joint ee: origin xyz=0.0001 -0.0205 -0.15 rpy=0 0 0 -> xyz=0.0001 -0.0205 -0.13 rpy=0 0 0
